File: ferrule-slot/eib-64-cap.kicad_sch (KiCad schematic)
At the start: 12 parts, among them J1 DF40C-70DP-0.4V(51), J10 DF40C-70DP-0.4V(51), J11 DF40C-70DP-0.4V(51), J12 DF40C-70DP-0.4V(51), J2 DF40C-70DP-0.4V(51), J3 DF40C-70DP-0.4V(51), J4 DF40C-70DP-0.4V(51), J5 DF40C-70DP-0.4V(51), J6 DF40C-70DP-0.4V(51), J7 DF40C-70DP-0.4V(51), J8 DF40C-70DP-0.4V(51), J9 DF40C-70DP-0.4V(51)

Commit message: Update to KiCAD 10 and prepare files for manufacturing
Parts:
- J1, J10, J11, J12, J2, J3, J4, J5, J6, J7, J8, J9: LCSC (none) -> C2692097; MPN (none) -> DF40C-70DP-0.4V(51); OEPS Description (none) -> CONNECTOR: HIROSE PLUG 70POS GOLD (OEPS M01 055) [DF40C-70D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; OEPS PN (none) -> OEPS070068
